File: bw16.kicad_pcb (KiCad board)
At the start: 2 copper layers, 30 x 57 mm, 27 parts, among them J1 Conn_01x08_Male, J2 Conn_01x08_Male, J3 Conn_01x08_Male, J4 Conn_01x08_Male, J5 Conn_01x03_Male, J6 +3V3, J7 GND, J8 VIN, M1 BW16, SW1 RESET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

Commit message: Add files via upload
Parts:
- added J9: Conn_01x06_Male, Connector_PinHeader_2.54mm:PinHeader_1x06_P2.54mm_Horizontal, F.Cu at (139.8, 133.0)
- moved J3 36.5 mm to (88.5, 74.5)
- moved J4 24.2 mm to (165.5, 88.5)
- moved C1 11.4 mm to (125.5, 122.5), turned to 180 degrees
- moved R2 4.12 mm to (139.5, 126.5)
- moved R4 3.50 mm to (127.5, 107.5)
- moved SW1 3.00 mm to (120.0, 118.0)
- moved R1 2.24 mm to (139.5, 124.0)
- moved R3 2.00 mm to (127.5, 104.5)
- moved J8 1.54 mm to (119.5, 126.0), turned to 180 degrees
- moved H4 1.00 mm to (145.0, 133.0)
- moved J7 0.72 mm to (136.1, 100.4)
- moved J6 0.61 mm to (127.6, 100.4)
- moved H2 0.25 mm to (121.8, 133.0)
Connections:
- D1 pad 1: Net-(D1-Pad1) -> /GND
- D3 pad 1: Net-(D3-Pad1) -> /GND
- J1 pad 3: Net-(J1-Pad3) -> /EN
- J2 pad 6: Net-(J2-Pad6) -> /PA12
- J3 pad 1: Net-(J1-Pad1) -> Net-(J3-Pad1)
- J3 pad 2: Net-(J1-Pad2) -> Net-(J3-Pad2)
- J3 pad 3: Net-(J1-Pad3) -> Net-(J3-Pad3)
- J3 pad 4: Net-(J1-Pad4) -> Net-(J3-Pad4)
- J3 pad 5: /LOG_RX -> Net-(J3-Pad5)
- J3 pad 6: Net-(J1-Pad6) -> Net-(J3-Pad6)
- J3 pad 7: Net-(J1-Pad7) -> Net-(J3-Pad7)
- J3 pad 8: /VDD33 -> Net-(J3-Pad8)
- J4 pad 1: /GND -> Net-(J4-Pad1)
- J4 pad 2: Net-(J2-Pad2) -> Net-(J4-Pad2)
- J4 pad 3: /LOG_TX -> Net-(J4-Pad3)
- J4 pad 4: Net-(J2-Pad4) -> Net-(J4-Pad4)
- J4 pad 5: Net-(J2-Pad5) -> Net-(J4-Pad5)
- J4 pad 6: Net-(J2-Pad6) -> Net-(J4-Pad6)
- J4 pad 7: Net-(J2-Pad7) -> Net-(J4-Pad7)
- J4 pad 8: Net-(J2-Pad8) -> Net-(J4-Pad8)
- J5 pad 1: /LOG_TX -> /GND
- J5 pad 3: /GND -> /LOG_TX
- M1 pad 14: Net-(J2-Pad6) -> /PA12
- M1 pad 3: Net-(J1-Pad3) -> /EN
- R3 pad 1: Net-(R3-Pad1) -> /VDD33
- R3 pad 2: Net-(R3-Pad2) -> Net-(D1-Pad2)
- R4 pad 1: Net-(R4-Pad1) -> /PA12
- R4 pad 2: Net-(R4-Pad2) -> Net-(D3-Pad2)
- SW1 pad 1: Net-(SW1-Pad1) -> /GND
- SW1 pad 2: Net-(SW1-Pad2) -> /EN
- SW2 pad 1: Net-(SW2-Pad1) -> /GND
- SW2 pad 2: Net-(SW2-Pad2) -> /LOG_TX
Routing:
- net /LOG_RX: track 2.87 -> 82.3 mm
- net /VDD33: track 7.35 -> 75.7 mm
- net /LOG_TX: track 3.10 -> 65.8 mm
- net /EN: track 0.00 -> 42.6 mm
- net /GND: track 7.19 -> 45.6 mm, vias 0 -> 26
- net /PA12: track 0.00 -> 34.1 mm
- net Net-(C1-Pad1): track 0.00 -> 14.5 mm
- net Net-(D3-Pad2): track 0.00 -> 10.4 mm
- net Net-(D1-Pad2): track 0.00 -> 9.66 mm
- net Net-(D2-Pad2): track 0.00 -> 4.46 mm
- net Net-(J1-Pad3): track 2.50 -> 0.00 mm
- net Net-(J2-Pad6): track 2.43 -> 0.00 mm
- net Net-(J2-Pad8): track 2.59 -> 4.74 mm
- net Net-(J2-Pad4): track 2.88 -> 4.71 mm
- net Net-(J1-Pad4): track 2.64 -> 4.45 mm
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- added copper zone on B.Cu, net /GND
- added copper zone on F.Cu, net /GND
Other:
- board size 30 x 57 mm -> 30.8 x 57 mm
- board text added: "0 PB2"
- board text added: "1 PB1"
- board text added: "14 PA7"
- board text added: "15 PA8"
- board text added: "16 PA25"
- board text added: "17 PA26"
- board text added: "18 PA15"
- board text added: "19 PA14"
- board text added: "2 PB3"
- board text added: "20 PA13"
- board text added: "21 PA12"
- board text added: "22 PA27"
- board text added: "23 PA30"
- board text added: "3V"
- board text added: "EN"
- board text added: "GND"
- board text added: "PA12"
- board text added: "RX"
- board text added: "TX"
- board text added: "VDD33"
- board text added: "Ver. 042221-31"
- board text added: "Vin"
- board text removed: "Ver. 30.2768"

Commit message: Add files via upload
Parts:
- moved J3 81.9 mm to (160.5, 113.5)
- moved J4 25.0 mm to (164.6, 113.5), turned to 0 degrees
- moved J5 10.0 mm to (156.0, 122.2)
- moved R1 3.61 mm to (142.5, 122.0)
- moved R2 3.61 mm to (142.5, 124.5)
- moved H3 1.00 mm to (145.0, 105.0)
- moved SW2 0.50 mm to (142.0, 118.0)
Connections:
- D2 pad 2: Net-(D2-Pad2) -> /VIN
- J5 pad 1: /GND -> Net-(J5-Pad1)
- J5 pad 2: /LOG_RX -> Net-(J5-Pad2)
- J5 pad 3: /LOG_TX -> Net-(J5-Pad3)
- J8 pad 1: Net-(D2-Pad2) -> /VIN
- J9 pad 2: /GND -> /EN
- J9 pad 5: Net-(J9-Pad5) -> /GND
- J9 pad 6: Net-(J9-Pad6) -> /VIN
Routing:
- net /EN: track 42.6 -> 67.5 mm, vias 0 -> 1
- net /VIN: track 0.00 -> 14.3 mm
- net /GND: track 45.6 -> 53.5 mm, vias 26 -> 25
- net /LOG_RX: track 82.3 -> 75.8 mm
- net Net-(D2-Pad2): track 4.46 -> 0.00 mm
- net /VDD33: track 75.7 -> 80.0 mm
- net /LOG_TX: track 65.8 -> 63.6 mm
- removed copper zone on B.Cu, net (none)
- removed copper zone on F.Cu, net (none)
Other:
- board text added: "-"
- board text added: ".."
- board text added: "5V"

Commit message: Add files via upload
add some text to make soldering more easy
Parts:
- removed J3, J4: Conn_01x08_Male, Connector_PinHeader_2.00mm:PinHeader_1x08_P2.00mm_Vertical
- removed J5: Conn_01x03_Male, Connector_PinHeader_2.54mm:PinHeader_1x03_P2.54mm_Vertical
Other:
- board text added: "10"
- board text added: "10K"
- board text added: "220"
- board text added: "47"
- board text added: "G"
- board text added: "Ham Check OK 2021.08.05"
- board text added: "JLCJLCJLCJLC"
- board text added: "R"
